Commit message: fix lidar tf

File: pinky_description/urdf/robot_core.xacro (robot description, xacro)
@@ -166,5 +166,5 @@
         <parent link="ydlidar_lidar_mount"/>
         <child link="laser_link"/>
-        <origin xyz="0.0 0 0.03" rpy="0 0 0"/>
+        <origin xyz="0.0 0 0.03" rpy="0 0 ${pi}"/>
     </joint>
 </robot>

Commit message: Fix typos and bugs

File: pinky_description/urdf/robot_core.xacro (robot description, xacro)
@@ -138,5 +138,5 @@
         <origin xyz="0.001 0 0.003" rpy="0 ${pi/2} 0"/>
     </joint>
-    <link name="ydlidar_lidar_mount">
+    <link name="rplidar_lidar_mount">
         <visual>
             <origin xyz="0 0 0" rpy="0 0 0"/>
@@ -157,12 +157,12 @@
         </inertial>
     </link>
-    <joint name="idar_mount_fixed_joint" type="fixed">
+    <joint name="lidar_mount_fixed_joint" type="fixed">
         <parent link="base_link"/>
-        <child link="ydlidar_lidar_mount"/>
+        <child link="rplidar_lidar_mount"/>
         <origin xyz="0 0 0.042" rpy="0 0 0"/>
     </joint>
     <link name="laser_link"/>
     <joint name="laser_link_fixed_joint" type="fixed">
-        <parent link="ydlidar_lidar_mount"/>
+        <parent link="rplidar_lidar_mount"/>
         <child link="laser_link"/>
         <origin xyz="0.0 0 0.03" rpy="0 0 ${pi}"/>

Commit message: update pinky nav2

File: pinky_description/urdf/robot_core.xacro (robot description, xacro)
@@ -168,3 +168,9 @@
         <origin xyz="0.0 0 0.03" rpy="0 0 ${pi}"/>
     </joint>
+    <link name="imu_link"/>
+    <joint name="imu_link_joint" type="fixed">
+        <parent link="base_link"/>
+        <child link="imu_link"/>
+        <origin xyz="0 0 0.03" rpy="0 0 0"/>
+    </joint>
 </robot>

Commit message: modify urdf

File: pinky_description/urdf/robot_core.xacro (robot description, xacro)
@@ -32,5 +32,5 @@
             <origin xyz="0 0 0" rpy="0 0 0"/>
             <geometry>
-                <mesh filename="package://pinky_description/meshes/visual/base_link_new.dae" scale="1 1 1"/>
+                <mesh filename="package://pinky_description/meshes/visual/base_link.dae" scale="1 1 1"/>
             </geometry>
         </visual>

Commit message: update gazebo pkg

File: pinky_description/urdf/robot_core.xacro (robot description, xacro)
@@ -134,5 +134,5 @@
     </link>
     <joint name="ul_sensor_mount_fixed_joint" type="fixed">
-        <parent link="base_link"/>
+        <parent link="chassis"/>
         <child link="ul_sensor_mount"/>
         <origin xyz="0.038 -0.002 -0.0035" rpy="0 0 0"/>
@@ -164,5 +164,5 @@
     </link>
     <joint name="front_camera_mount_fixed_joint" type="fixed">
-        <parent link="base_link"/>
+        <parent link="chassis"/>
         <child link="front_camera_mount"/>
         <origin xyz="0.05 -0.001 0.028" rpy="0 0 0"/>
@@ -174,5 +174,5 @@
         <origin xyz="0.001 0 0.003" rpy="0 0 0"/>
     </joint>
-    <link name="rplidar_lidar_mount">
+    <link name="lidar_lidar_mount">
         <visual>
             <origin xyz="0 0 0" rpy="0 0 0"/>
@@ -194,11 +194,11 @@
     </link>
     <joint name="lidar_mount_fixed_joint" type="fixed">
-        <parent link="base_link"/>
-        <child link="rplidar_lidar_mount"/>
+        <parent link="chassis"/>
+        <child link="lidar_lidar_mount"/>
         <origin xyz="0 0 0.042" rpy="0 0 0"/>
     </joint>
     <link name="laser_link"/>
     <joint name="laser_link_fixed_joint" type="fixed">
-        <parent link="rplidar_lidar_mount"/>
+        <parent link="lidar_lidar_mount"/>
         <child link="laser_link"/>
         <origin xyz="0.0 0 0.03" rpy="0 0 ${pi}"/>
@@ -213,5 +213,5 @@
     </link>
     <joint name="imu_link_joint" type="fixed">
-        <parent link="base_link"/>
+        <parent link="chassis"/>
         <child link="imu_link"/>
         <origin xyz="0 0 0.03" rpy="0 0 0"/>

Commit message: modify camera tf

File: pinky_description/urdf/robot_core.xacro (robot description, xacro)
@@ -172,5 +172,5 @@
         <parent link="front_camera_mount"/>
         <child link="camera_link"/>
-        <origin xyz="0.001 0 0.003" rpy="0 0 0"/>
+        <origin xyz="0.001 0 0.003" rpy="-${pi/2} 0 -${pi/2}"/>
     </joint>
     <link name="lidar_lidar_mount">
