Commit message: update pinky gazebo

File: pinky_description/urdf/camera.xacro (robot description, xacro)
@@ -3,7 +3,11 @@
     <gazebo reference="camera_link">
         <sensor name="camera" type="camera">
-            <update_rate>30.0</update_rate>
-            <camera name="camera">
-                <pose>0 0 0 0 -1.5707 0</pose>
+            <always_on>true</always_on>
+            <visualize>true</visualize>
+            <update_rate>30</update_rate>
+            <topic>camera/image_raw</topic>
+            <gz_frame_id>camera_rgb_frame</gz_frame_id>
+            <camera name="intel_realsense_r200">
+                <camera_info_topic>camera/camera_info</camera_info_topic>
                 <horizontal_fov>1.08</horizontal_fov>
                 <image>
@@ -22,8 +26,4 @@
                 </noise>
             </camera>
-            <plugin name="camera_controller" filename="libgazebo_ros_camera.so">
-                <frame_name>camera_link</frame_name>
-                <hack_baseline>0.07</hack_baseline>
-            </plugin>
         </sensor>
     </gazebo>

File: pinky_description/urdf/gazebo_control.xacro (robot description, xacro)
@@ -2,19 +2,21 @@
 <robot xmlns:xacro="http://www.ros.org/wiki/xacro">
     <gazebo>
-        <plugin name="diff_drive" filename="libgazebo_ros_diff_drive.so">
-            <!-- Wheel Information -->
+        <plugin filename="gz-sim-diff-drive-system" name="gz::sim::systems::DiffDrive">
             <left_joint>left_wheel_joint</left_joint>
             <right_joint>right_wheel_joint</right_joint>
             <wheel_separation>0.11</wheel_separation>
-            <wheel_diameter>0.06</wheel_diameter>
-            <!-- Limits -->
-            <max_wheel_torque>200</max_wheel_torque>
-            <max_wheel_acceleration>0.25</max_wheel_acceleration>
-            <!-- Output -->
-            <odometry_frame>odom</odometry_frame>
-            <robot_base_frame>base_link</robot_base_frame>
-            <publish_odom>false</publish_odom>
-            <publish_odom_tf>false</publish_odom_tf>
-            <publish_wheel_tf>true</publish_wheel_tf>
+            <wheel_radius>0.06</wheel_radius>
+            <max_linear_acceleration>0.5</max_linear_acceleration>
+            <topic>cmd_vel</topic>
+            <odom_topic>odom</odom_topic>
+            <frame_id>odom</frame_id>
+            <child_frame_id>base_footprint</child_frame_id>
+            <odom_publisher_frequency>30</odom_publisher_frequency>
+            <tf_topic>/tf</tf_topic>
+        </plugin>
+        <plugin filename="gz-sim-joint-state-publisher-system" name="gz::sim::systems::JointStatePublisher">
+            <topic>joint_states</topic>
+            <joint_name>left_wheel_joint</joint_name>
+            <joint_name>right_wheel_joint</joint_name>
         </plugin>
     </gazebo>

File: pinky_description/urdf/lidar.xacro (robot description, xacro)
@@ -2,13 +2,15 @@
 <robot xmlns:xacro="http://www.ros.org/wiki/xacro" >
     <gazebo reference="laser_link">
-        <sensor name="laser" type="ray">
-            <pose>0 0 0 0 0 0</pose>
-            <always_on>1</always_on>
-            <update_rate>15</update_rate>
-            <visualize>false</visualize>
-            <ray>
+        <sensor name="laser" type="gpu_lidar">
+            <always_on>true</always_on>
+            <visualize>true</visualize>
+            <pose> 0 0 0 0 0 0 </pose>
+            <update_rate>5</update_rate>
+            <topic>scan</topic>
+            <gz_frame_id>laser_link</gz_frame_id>
+            <lidar>
                 <scan>
                     <horizontal>
-                        <samples>375</samples>
+                        <samples>360</samples>
                         <resolution>1</resolution>
                         <min_angle>${-180*pi/180}</min_angle>
@@ -26,12 +28,5 @@
                     <stddev>0.01</stddev>
                 </noise>
-            </ray>
-            <plugin name="laser" filename="libgazebo_ros_ray_sensor.so">
-                <ros>
-                    <remapping>~/out:=scan</remapping>
-                </ros>
-                <frame_name>laser_link</frame_name>
-                <output_type>sensor_msgs/LaserScan</output_type>
-            </plugin>
+            </lidar>
         </sensor>
     </gazebo>

File: pinky_description/urdf/robot.urdf.xacro (robot description, xacro)
@@ -1,8 +1,8 @@
 <?xml version="1.0"?>
-<robot name="my_mobile" xmlns:xacro="http://www.ros.org/wiki/xacro">
+<robot name="pinky" xmlns:xacro="http://www.ros.org/wiki/xacro">
     <xacro:include filename="robot_core.xacro"/>
     <xacro:include filename="robot_gazebo.xacro"/>
-    <!-- <xacro:include filename="gazebo_control.xacro"/> -->
-    <xacro:include filename="ros2_control.xacro" />
+    <xacro:include filename="gazebo_control.xacro"/>
+    <!-- <xacro:include filename="ros2_control.xacro" /> -->
     <xacro:include filename="lidar.xacro" />
     <xacro:include filename="camera.xacro"/>

File: pinky_description/urdf/robot_core.xacro (robot description, xacro)
@@ -1,6 +1,19 @@
 <?xml version="1.0"?>
-<robot name="my_mobile" xmlns:xacro="http://www.ros.org/wiki/xacro">
+<robot name="pinky" xmlns:xacro="http://www.ros.org/wiki/xacro">
     <xacro:property name="wheel_separation" value="0.1"/>
     <xacro:property name="wheel_diameter" value="0.06"/>
+    <xacro:include filename="inertial_macros.xacro"/>
+    <xacro:property name="chassis_length" value="0.10"/>
+    <xacro:property name="chassis_width" value="0.08"/>
+    <xacro:property name="chassis_height" value="0.06"/>
+    <xacro:property name="chassis_mass" value="1.0"/>
+    <xacro:property name="wheel_radius" value="0.03"/>
+    <xacro:property name="wheel_thickness" value="0.014"/>
+    <xacro:property name="wheel_mass" value="0.05"/>
+    <xacro:property name="caster_wheel_radius" value="0.01"/>
+    <xacro:property name="caster_wheel_mass" value="0.7"/>
+    <material name="white">
+        <color rgba="1 1 1 1" />
+    </material>
     <link name="base_footprint"/>
     <joint name="base_link_fixed_joint" type="fixed">
@@ -9,23 +22,50 @@
         <origin xyz="0 0 ${wheel_diameter/2}" rpy="0 0 0"/>
     </joint>
-	<link name="base_link">
+	<link name="base_link"/>
+     <joint name="chassis_fixed_joint" type="fixed">
+        <parent link="base_link"/>
+        <child link="chassis"/>
+        <origin xyz="0 0 0" rpy="0 0 0"/>
+    </joint>
+	<link name="chassis">
 		<visual>
             <origin xyz="0 0 0" rpy="0 0 0"/>
             <geometry>
-                <mesh filename="package://pinky_description/meshes/visual/base_link.dae" scale="1 1 1"/>
-            </geometry>
-        </visual>
-        <collision>
-            <origin xyz="0 0 0" rpy="0 0 0"/>
-            <geometry>
-                <mesh filename="package://pinky_description/meshes/collision/base_link.stl" scale="1 1 1"/>
-            </geometry>
-        </collision>
-        <inertial>
-            <origin xyz="-0.02 0 0.028" rpy="0 0 0"/>
-            <mass value="0.5"/>
-            <inertia ixx="0.01" ixy="0" ixz="0" iyy="0.01" iyz="0" izz="0.01"/>
-        </inertial>
+                <mesh filename="package://pinky_description/meshes/visual/base_link_new.dae" scale="1 1 1"/>
+            </geometry>
+        </visual>
+        <collision>
+            <origin xyz="-0.01 0 0.01" rpy="0 0 0"/>
+            <geometry>
+                <box size="${chassis_length} ${chassis_width} ${chassis_height}"/>
+            </geometry>
+        </collision>
+        <xacro:inertial_box mass="${chassis_mass}" x="${chassis_length}" y="${chassis_width}" z="${chassis_height}">
+            <origin xyz="-0.01 0 0.01" rpy="0 0 0"/>
+        </xacro:inertial_box>
 	</link>
+    <joint name="caster_fixed_joint" type="fixed">
+        <parent link="chassis"/>
+        <child link="caster"/>
+        <origin xyz="-0.044 0 -0.02" rpy="0 0 0"/>
+    </joint>
+	<link name="caster">
+      <visual>
+            <origin xyz="0 0 0" rpy="0 0 0"/>
+            <geometry>
+                <sphere radius="${caster_wheel_radius}"/>
+            </geometry>
+            <material name="white"/>
+        </visual>
+        <collision>
+            <origin xyz="0 0 0" rpy="0 0 0"/>
+            <geometry>
+                <sphere radius="${caster_wheel_radius}"/>
+            </geometry>
+        </collision>
+        <xacro:inertial_sphere mass="${caster_wheel_mass}" radius="${caster_wheel_radius}">
+            <origin xyz="0 0 0" rpy="0 0 0"/>
+        </xacro:inertial_sphere>
+    </link>
     <joint name="left_wheel_joint" type="continuous">
         <parent link="base_link"/>
@@ -44,12 +84,10 @@
             <origin xyz="0 0 0" rpy="0 0 0"/>
             <geometry>
-                <mesh filename="package://pinky_description/meshes/collision/wheel.stl" scale="1 1 1"/>
-            </geometry>
-        </collision>
-        <inertial>
-            <origin xyz="0 0 0" rpy="0 0 0"/>
-            <mass value="0.3"/>
-            <inertia ixx="0.1" ixy="0" ixz="0" iyy="0.1" iyz="0" izz="0.1"/>
-        </inertial>
+                <cylinder radius="${wheel_radius}" length="${wheel_thickness}"/>
+            </geometry>
+        </collision>
+        <xacro:inertial_cylinder mass="${wheel_mass}" length="${wheel_thickness}" radius="${wheel_radius}">
+            <origin xyz="0 0 0" rpy="0 0 0"/>
+        </xacro:inertial_cylinder>
     </link>
     <joint name="right_wheel_joint" type="continuous">
@@ -69,12 +107,10 @@
             <origin xyz="0 0 0" rpy="0 0 0"/>
             <geometry>
-                <mesh filename="package://pinky_description/meshes/collision/wheel.stl" scale="1 1 1"/>
-            </geometry>
-        </collision>
-        <inertial>
-            <origin xyz="0 0 0" rpy="0 0 0"/>
-            <mass value="0.3"/>
-            <inertia ixx="0.1" ixy="0" ixz="0" iyy="0.1" iyz="0" izz="0.1"/>
-        </inertial>
+                <cylinder radius="${wheel_radius}" length="${wheel_thickness}"/>
+            </geometry>
+        </collision>
+        <xacro:inertial_cylinder mass="${wheel_mass}" length="${wheel_thickness}" radius="${wheel_radius}">
+            <origin xyz="0 0 0" rpy="0 0 0"/>
+        </xacro:inertial_cylinder>
     </link>
     <link name="ul_sensor_mount">
@@ -136,5 +172,5 @@
         <parent link="front_camera_mount"/>
         <child link="camera_link"/>
-        <origin xyz="0.001 0 0.003" rpy="0 ${pi/2} 0"/>
+        <origin xyz="0.001 0 0.003" rpy="0 0 0"/>
     </joint>
     <link name="rplidar_lidar_mount">
@@ -168,5 +204,12 @@
         <origin xyz="0.0 0 0.03" rpy="0 0 ${pi}"/>
     </joint>
-    <link name="imu_link"/>
+    <link name="imu_link">
+        <sensor name="imu_sensor" type="imu">
+            <always_on>1</always_on>
+            <update_rate>1</update_rate>
+            <visualize>true</visualize>
+            <topic>imu</topic>
+        </sensor>
+    </link>
     <joint name="imu_link_joint" type="fixed">
         <parent link="base_link"/>

File: pinky_description/urdf/robot_gazebo.xacro (robot description, xacro)
@@ -1,19 +1,22 @@
 <?xml version="1.0"?>
-<robot name="my_mobile" xmlns:xacro="http://www.ros.org/wiki/xacro">
+<robot name="pinky" xmlns:xacro="http://www.ros.org/wiki/xacro">
     <gazebo reference="left_wheel">
-        <mu1>200</mu1>
-        <mu2>200</mu2>
-        <kp>10000000.0</kp>
-        <kd>1.0</kd>
+        <selfCollide>false</selfCollide>
+            <mu1 value="1.2" />
+            <mu2 value="1.2" />
     </gazebo>
     <gazebo reference="right_wheel">
-        <mu1>200</mu1>
-        <mu2>200</mu2>
-        <kp>10000000.0</kp>
-        <kd>1.0</kd>
+        <selfCollide>false</selfCollide>
+            <mu1 value="1.2" />
+            <mu2 value="1.2" />
     </gazebo>
     <gazebo reference="base_link">
-        <mu1>0.0</mu1>
-        <mu2>0.0</mu2>
+	  <selfCollide>false</selfCollide>
+      <mu1 value="0.05" />
+      <mu2 value="0.05" />
+    </gazebo>
+    <gazebo reference="caster">
+      <mu1 value="0.05" />
+      <mu2 value="0.05" />
     </gazebo>
 </robot>

File: pinky_description/urdf/ros2_control.xacro (robot description, xacro)
@@ -1,7 +1,7 @@
 <?xml version="1.0"?>
 <robot xmlns:xacro="http://www.ros.org/wiki/xacro">
-    <ros2_control name="my_robot_system" type="system">
+    <ros2_control name="GazeboSimSystem" type="system">
         <hardware>
-            <plugin>gazebo_ros2_control/GazeboSystem</plugin>
+            <plugin>gz_ros2_control/GazeboSimSystem</plugin>
         </hardware>
         <joint name="left_wheel_joint">
@@ -23,8 +23,8 @@
     </ros2_control>
     <gazebo>
-        <plugin filename="libgazebo_ros2_control.so" name="gazebo_ros2_control">
+        <plugin filename="gz_ros2_control-system" name="gz_ros2_control::GazeboSimROS2ControlPlugin">
             <parameters>$(find pinky_gazebo)/config/my_controllers.yaml</parameters>
             <ros>
-                <remapping>diff_cont/cmd_vel_unstamped:=cmd_vel</remapping>
+                <remapping>diff_cont/cmd_vel:=cmd_vel</remapping>
                 <remapping>diff_cont/odom:=odom</remapping>
             </ros>

Commit message: update gazebo pkg

File: pinky_description/urdf/camera.xacro (robot description, xacro)
@@ -3,4 +3,5 @@
     <gazebo reference="camera_link">
         <sensor name="camera" type="camera">
+            <pose>0 0 0 0 -1.5708 1.5708</pose>
             <always_on>true</always_on>
             <visualize>true</visualize>
@@ -8,5 +9,5 @@
             <topic>camera/image_raw</topic>
             <gz_frame_id>camera_rgb_frame</gz_frame_id>
-            <camera name="intel_realsense_r200">
+            <camera name="pinky_camera">
                 <camera_info_topic>camera/camera_info</camera_info_topic>
                 <horizontal_fov>1.08</horizontal_fov>

File: pinky_description/urdf/gazebo_control.xacro (robot description, xacro)
@@ -5,7 +5,10 @@
             <left_joint>left_wheel_joint</left_joint>
             <right_joint>right_wheel_joint</right_joint>
-            <wheel_separation>0.11</wheel_separation>
-            <wheel_radius>0.06</wheel_radius>
-            <max_linear_acceleration>0.5</max_linear_acceleration>
+            <wheel_separation>0.096</wheel_separation>
+            <wheel_radius>0.03</wheel_radius>
+            <min_velocity>-0.5</min_velocity>
+            <max_velocity>0.5</max_velocity>
+            <min_acceleration>-2.0</min_acceleration>
+            <max_acceleration>2.0</max_acceleration>
             <topic>cmd_vel</topic>
             <odom_topic>odom</odom_topic>

File: pinky_description/urdf/robot.urdf.xacro (robot description, xacro)
@@ -2,8 +2,8 @@
 <robot name="pinky" xmlns:xacro="http://www.ros.org/wiki/xacro">
     <xacro:include filename="robot_core.xacro"/>
+    <xacro:include filename="lidar.xacro" />
+    <xacro:include filename="camera.xacro"/>
+    <xacro:include filename="imu.xacro"/>
     <xacro:include filename="robot_gazebo.xacro"/>
     <xacro:include filename="gazebo_control.xacro"/>
-    <!-- <xacro:include filename="ros2_control.xacro" /> -->
-    <xacro:include filename="lidar.xacro" />
-    <xacro:include filename="camera.xacro"/>
 </robot>

File: pinky_description/urdf/robot_core.xacro (robot description, xacro)
@@ -1,5 +1,5 @@
 <?xml version="1.0"?>
 <robot name="pinky" xmlns:xacro="http://www.ros.org/wiki/xacro">
-    <xacro:property name="wheel_separation" value="0.1"/>
+    <xacro:property name="wheel_separation" value="0.11"/>
     <xacro:property name="wheel_diameter" value="0.06"/>
     <xacro:include filename="inertial_macros.xacro"/>
@@ -204,12 +204,5 @@
         <origin xyz="0.0 0 0.03" rpy="0 0 ${pi}"/>
     </joint>
-    <link name="imu_link">
-        <sensor name="imu_sensor" type="imu">
-            <always_on>1</always_on>
-            <update_rate>1</update_rate>
-            <visualize>true</visualize>
-            <topic>imu</topic>
-        </sensor>
-    </link>
+    <link name="imu_link"/>
     <joint name="imu_link_joint" type="fixed">
         <parent link="chassis"/>

File: pinky_description/urdf/robot_gazebo.xacro (robot description, xacro)
@@ -2,21 +2,18 @@
 <robot name="pinky" xmlns:xacro="http://www.ros.org/wiki/xacro">
     <gazebo reference="left_wheel">
-        <selfCollide>false</selfCollide>
-            <mu1 value="1.2" />
-            <mu2 value="1.2" />
+      <mu1 value="1.2" />
+      <mu2 value="1.2" />
     </gazebo>
     <gazebo reference="right_wheel">
-        <selfCollide>false</selfCollide>
-            <mu1 value="1.2" />
-            <mu2 value="1.2" />
+      <mu1 value="1.2" />
+      <mu2 value="1.2" />
     </gazebo>
     <gazebo reference="base_link">
-	  <selfCollide>false</selfCollide>
-      <mu1 value="0.05" />
-      <mu2 value="0.05" />
+      <mu1 value="0.01" />
+      <mu2 value="0.01" />
     </gazebo>
     <gazebo reference="caster">
-      <mu1 value="0.05" />
-      <mu2 value="0.05" />
+      <mu1 value="0.01" />
+      <mu2 value="0.01" />
     </gazebo>
 </robot>
